Commit message: git subrepo pull --branch=public_release ros2
subrepo:
  subdir:   "ros2"
  merged:   "d4283ae"
upstream:
  origin:   "https://github.com/TetherIA/aero-open-ros2.git"
  branch:   "public_release"
  commit:   "d4283ae"
git-subrepo:
  version:  "0.4.9"
  origin:   "https://github.com/Homebrew/brew"
  commit:   "490e51d47f"

File: ros2/src/aero_hand_open_description/urdf/aero_hand_open_left.urdf (robot description, URDF)
Before this commit: robot aero_hand_open_left, 22 links, 21 joints
Joints:
- joint left_index_dip: axis -1 -0 -0 -> 1 1.224646799e-16 0; origin xyz=0 0 0.022 rpy=0 -0 0 -> xyz=0 0 0.022 rpy=0 -0 -4.102069795e-10
- joint left_index_mcp_flex: axis -1 -0 -0 -> 1 1.224646799e-16 0; origin xyz=0.030626 0.0011782 0.10542 rpy=0 0.05236 0.034907 -> xyz=-0.030626 -0.0011782 0.10542 rpy=6.418116951e-18 -0.05236 0.03490699959
- joint left_index_pip: axis -1 -0 -0 -> 1 1.224646799e-16 0; origin xyz=0 0.0014554 0.043 rpy=0 -0 0 -> xyz=1.782350951e-19 -0.0014554 0.043 rpy=0 -0 -4.102069795e-10
- joint left_index_tip: axis -0 -0 -0 -> 0 0 0; origin xyz=0 -0.003512 0.026776 rpy=0 -0 0 -> xyz=-4.300959559e-19 0.003512 0.026776 rpy=0 -0 -4.102069795e-10
- joint left_middle_dip: axis -1 -0 -0 -> 1 1.224646799e-16 0; origin xyz=0 0 0.022 rpy=0 -0 0 -> xyz=0 0 0.022 rpy=0 -0 -4.102069795e-10
- joint left_middle_mcp_flex: axis -1 -0 -0 -> 1 1.224646799e-16 0; origin xyz=0.0075 0 0.106 rpy=0 -0 0 -> xyz=-0.0075 -9.184850994e-19 0.106 rpy=0 -0 4.102069795e-10
- joint left_middle_pip: axis -1 -0 -0 -> 1 1.224646799e-16 0; origin xyz=0 0.0014554 0.043 rpy=0 -0 0 -> xyz=1.782350951e-19 -0.0014554 0.043 rpy=0 -0 -4.102069795e-10
- joint left_middle_tip: axis -0 -0 -0 -> 0 0 0; origin xyz=0 -0.003512 0.026776 rpy=0 -0 0 -> xyz=-4.300959559e-19 0.003512 0.026776 rpy=0 -0 -4.102069795e-10
- joint left_pinky_dip: axis -1 -0 -0 -> 1 1.224646799e-16 0; origin xyz=0 0 0.022 rpy=0 -0 0 -> xyz=0 0 0.022 rpy=0 -0 -4.102069795e-10
- joint left_pinky_mcp_flex: axis -1 -0 -0 -> 1 1.224646799e-16 0; origin xyz=-0.038266 0.0036416 0.092393 rpy=0 -0.10472 -0.069946 -> xyz=0.038266 -0.0036416 0.092393 rpy=-1.287158685e-17 0.10472 -0.06994599959
- joint left_pinky_pip: axis -1 -0 -0 -> 1 1.224646799e-16 0; origin xyz=0 0.0014554 0.043 rpy=0 -0 0 -> xyz=1.782350951e-19 -0.0014554 0.043 rpy=0 -0 -4.102069795e-10
- joint left_pinky_tip: axis -0 -0 -0 -> 0 0 0; origin xyz=0 -0.003512 0.026776 rpy=0 -0 0 -> xyz=-4.300959559e-19 0.003512 0.026776 rpy=0 -0 -4.102069795e-10
- joint left_ring_dip: axis -1 -0 -0 -> 1 1.224646799e-16 0; origin xyz=0 0 0.022 rpy=0 -0 0 -> xyz=0 0 0.022 rpy=0 -0 -4.102069795e-10
- joint left_ring_mcp_flex: axis -1 -0 -0 -> 1 1.224646799e-16 0; origin xyz=-0.015626 0.0011782 0.10542 rpy=0 -0.05236 -0.034907 -> xyz=0.015626 -0.0011782 0.10542 rpy=-6.418116951e-18 0.05236 -0.03490699959
- joint left_ring_pip: axis -1 -0 -0 -> 1 1.224646799e-16 0; origin xyz=0 0.0014554 0.043 rpy=0 -0 0 -> xyz=1.782350951e-19 -0.0014554 0.043 rpy=0 -0 -4.102069795e-10
- joint left_ring_tip: axis -0 -0 -0 -> 0 0 0; origin xyz=0 -0.003512 0.026776 rpy=0 -0 0 -> xyz=-4.300959559e-19 0.003512 0.026776 rpy=0 -0 -4.102069795e-10
- joint left_thumb_cmc_abd: axis -0 1 -0 -> 1.224646799e-16 -1 0; origin xyz=0.028112 0.0145 0.025363 rpy=1.2217 -0 1.57 -> xyz=-0.028112 -0.0145 0.025363 rpy=-1.2217 -1.150778795e-16 1.57
- joint left_thumb_cmc_flex: axis -1 -0 -0 -> 1 1.224646799e-16 0; origin xyz=-0.003475 -0.003808 0.019656 rpy=-0.1325 -0.17906 -0.26195 -> xyz=0.003475 0.003808 0.019656 rpy=0.1325 0.17906 -0.2619499996
- joint left_thumb_ip: axis -1 -0 -0 -> 1 1.224646799e-16 0; origin xyz=0 -0.002206 0.029919 rpy=0 -0 0 -> xyz=-2.701570839e-19 0.002206 0.029919 rpy=0 -0 -4.102069795e-10
- joint left_thumb_mcp: axis -1 -0 -0 -> 1 1.224646799e-16 0; origin xyz=0 -0.0033822 0.035848 rpy=0 -0 0 -> xyz=-4.142000404e-19 0.0033822 0.035848 rpy=0 -0 -4.102069795e-10
- joint left_thumb_tip: axis -0 -0 -0 -> 0 0 0; origin xyz=0 -0.0059474 0.031823 rpy=0 -0 0 -> xyz=-7.283464373e-19 0.0059474 0.031823 rpy=0 -0 -4.102069795e-10

Commit message: git subrepo pull --branch=public_release --force ros2
subrepo:
  subdir:   "ros2"
  merged:   "26392bf"
upstream:
  origin:   "https://github.com/TetherIA/aero-open-ros2.git"
  branch:   "public_release"
  commit:   "26392bf"
git-subrepo:
  version:  "0.4.9"
  origin:   "https://github.com/ingydotnet/git-subrepo"
  commit:   "6232cc5"

File: ros2/src/aero_hand_open_description/urdf/aero_hand_open_left.urdf (robot description, URDF)
Before this commit: robot aero_hand_open_left, 22 links, 21 joints
Joints:
- joint left_index_dip: axis 1 1.224646799e-16 0 -> -1 0 0; origin xyz=0 0 0.022 rpy=0 -0 -4.102069795e-10 -> xyz=0 0 0.022 rpy=0 0 0
- joint left_index_mcp_flex: axis 1 1.224646799e-16 0 -> -1 0 0; origin xyz=-0.030626 -0.0011782 0.10542 rpy=6.418116951e-18 -0.05236 0.03490699959 -> xyz=-0.030626 -0.0011782 0.10542 rpy=0 -0.05236 0.034907
- joint left_index_pip: axis 1 1.224646799e-16 0 -> -1 0 0; origin xyz=1.782350951e-19 -0.0014554 0.043 rpy=0 -0 -4.102069795e-10 -> xyz=0 -0.0014554 0.043 rpy=0 0 0
- joint left_index_tip: origin xyz=-4.300959559e-19 0.003512 0.026776 rpy=0 -0 -4.102069795e-10 -> xyz=0 0.003512 0.026776 rpy=0 0 0
- joint left_middle_dip: axis 1 1.224646799e-16 0 -> -1 0 0; origin xyz=0 0 0.022 rpy=0 -0 -4.102069795e-10 -> xyz=0 0 0.022 rpy=0 0 0
- joint left_middle_mcp_flex: axis 1 1.224646799e-16 0 -> -1 0 0; origin xyz=-0.0075 -9.184850994e-19 0.106 rpy=0 -0 4.102069795e-10 -> xyz=-0.0075 0 0.106 rpy=0 0 0
- joint left_middle_pip: axis 1 1.224646799e-16 0 -> -1 0 0; origin xyz=1.782350951e-19 -0.0014554 0.043 rpy=0 -0 -4.102069795e-10 -> xyz=0 -0.0014554 0.043 rpy=0 0 0
- joint left_middle_tip: origin xyz=-4.300959559e-19 0.003512 0.026776 rpy=0 -0 -4.102069795e-10 -> xyz=0 0.003512 0.026776 rpy=0 0 0
- joint left_pinky_dip: axis 1 1.224646799e-16 0 -> -1 0 0; origin xyz=0 0 0.022 rpy=0 -0 -4.102069795e-10 -> xyz=0 0 0.022 rpy=0 0 0
- joint left_pinky_mcp_flex: axis 1 1.224646799e-16 0 -> -1 0 0; origin xyz=0.038266 -0.0036416 0.092393 rpy=-1.287158685e-17 0.10472 -0.06994599959 -> xyz=0.038266 -0.0036416 0.092393 rpy=0 0.10472 -0.069946
- joint left_pinky_pip: axis 1 1.224646799e-16 0 -> -1 0 0; origin xyz=1.782350951e-19 -0.0014554 0.043 rpy=0 -0 -4.102069795e-10 -> xyz=0 -0.0014554 0.043 rpy=0 0 0
- joint left_pinky_tip: origin xyz=-4.300959559e-19 0.003512 0.026776 rpy=0 -0 -4.102069795e-10 -> xyz=0 0.003512 0.026776 rpy=0 0 0
- joint left_ring_dip: axis 1 1.224646799e-16 0 -> -1 0 0; origin xyz=0 0 0.022 rpy=0 -0 -4.102069795e-10 -> xyz=0 0 0.022 rpy=0 0 0
- joint left_ring_mcp_flex: axis 1 1.224646799e-16 0 -> -1 0 0; origin xyz=0.015626 -0.0011782 0.10542 rpy=-6.418116951e-18 0.05236 -0.03490699959 -> xyz=0.015626 -0.0011782 0.10542 rpy=0 0.05236 -0.034907
- joint left_ring_pip: axis 1 1.224646799e-16 0 -> -1 0 0; origin xyz=1.782350951e-19 -0.0014554 0.043 rpy=0 -0 -4.102069795e-10 -> xyz=0 -0.0014554 0.043 rpy=0 0 0
- joint left_ring_tip: origin xyz=-4.300959559e-19 0.003512 0.026776 rpy=0 -0 -4.102069795e-10 -> xyz=0 0.003512 0.026776 rpy=0 0 0
- joint left_thumb_cmc_abd: axis 1.224646799e-16 -1 0 -> 0 1 0; origin xyz=-0.028112 -0.0145 0.025363 rpy=-1.2217 -1.150778795e-16 1.57 -> xyz=-0.028112 -0.0145 0.025363 rpy=-1.2217 0 1.57
- joint left_thumb_cmc_flex: axis 1 1.224646799e-16 0 -> -1 0 0; origin xyz=0.003475 0.003808 0.019656 rpy=0.1325 0.17906 -0.2619499996 -> xyz=0.003475 0.003808 0.019656 rpy=0.1325 0.17906 -0.26195
- joint left_thumb_ip: axis 1 1.224646799e-16 0 -> -1 0 0; origin xyz=-2.701570839e-19 0.002206 0.029919 rpy=0 -0 -4.102069795e-10 -> xyz=0 0.002206 0.029919 rpy=0 0 0
- joint left_thumb_mcp: axis 1 1.224646799e-16 0 -> -1 0 0; origin xyz=-4.142000404e-19 0.0033822 0.035848 rpy=0 -0 -4.102069795e-10 -> xyz=0 0.0033822 0.035848 rpy=0 0 0
- joint left_thumb_tip: origin xyz=-7.283464373e-19 0.0059474 0.031823 rpy=0 -0 -4.102069795e-10 -> xyz=0 0.0059474 0.031823 rpy=0 0 0
